File: Motor_Controllers.kicad_sch (KiCad schematic)
At the start: 16 parts, among them J4 Conn_01x06_Socket, J5 Conn_01x06_Socket, U3 DRV8874_Carrier, U4 DRV8874_Carrier

Commit message: Started with routing
Parts:
- J4: value Conn_01x06_Socket -> MOT-A
- J5: value Conn_01x06_Socket -> MOT-B
Changed lines of the file:
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@@
 			)
 		)
-		(property "Value" "Conn_01x06_Socket"
+		(property "Value" "MOT-B"
 			(at 238.76 72.39 0)
 			(effects
@@
 			)
 		)
-		(property "Value" "Conn_01x06_Socket"
+		(property "Value" "MOT-A"
 			(at 109.855 50.8 0)
 			(effects
