File: BalancingRobot_Teensy41.kicad_sch (KiCad schematic)
At the start: 6 parts, among them J1 PM02D, J2 UART, J3 XT30, U1 Teensy4.1

Commit message: Almost completed with routing
Parts:
- added H1, H2, H3, H4: MountingHole_Pad, MountingHole:MountingHole_3.2mm_M3_Pad_Via, symbol Mechanical:MountingHole_Pad
Connections:
- net GND: now also H1.1, H2.1, H3.1, H4.1
- no-connect marks 39 -> 21
